File: AudioVisualizer/boardSchematic.brd (EAGLE design)
At the start: 128 x 65 mm, 84 parts

Commit message: Finished board layout
Routing:
- net GND: track 93.3 -> 95.0 mm
Other:
- board text added: "Designed by Zach Kauffman & Isaac Rex"
- board text added: "IN"
- board text added: "OUT"
